File: RC Light System Output/Ports.sch (KiCad schematic (older format))
At the start: 36 parts, among them J10 EX_B, J3 FL_A, J4 FL_B, J5 BR_A, J6 BR_B, J7 BL_L, J8 BL_R, J9 EX_A, Q1 2N2222, Q2 2N2222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

Commit message: Map footprints and add transistor pulldowns
Parts:
- added RN1: 10k, Resistor_THT:R_Array_SIP9, symbol Device:R_Network08
- J10, J3, J4, J5, J6, J7, J8, J9: footprint (none) -> Connector_JST:JST_XH_B2B-XH-A_1x02_P2.50mm_Vertical
- JP1, JP2, JP3, JP4: footprint (none) -> solder_bridge:bridge_open
- Q1, Q2, Q3, Q4, Q5, Q6, Q7, Q8: footprint Package_TO_SOT_THT:TO-92_Inline -> Package_TO_SOT_THT:TO-92_HandSolder
- R1, R10, R11, R12, R13, R15, R2, R3, R4, R5, R6, R7, R8, R9: footprint (none) -> resistor:R_Axial_DIN0207_L6.3mm_D2.5mm_P7.62mm_Horizontal
- R14, R16: value 4k7 -> 10; footprint (none) -> resistor:R_Axial_DIN0207_L6.3mm_D2.5mm_P7.62mm_Horizontal
Connections:
- net BL_L: now also RN1.6 (R5)
- net BL_R: now also RN1.7 (R6)
- net BR_A: now also RN1.4 (R3)
- net BR_B: now also RN1.5 (R4)
- net EX_A: now also RN1.8 (R7)
- net EX_B: now also RN1.9 (R8)
- net FL_A: now also RN1.2 (R1)
- net FL_B: now also RN1.3 (R2)
- net GND: now also RN1.1 (common)
Other:
- note added: "Assuming LEDs with resistors already\nin the lead, resistor as failsafe."

Commit message: First layout done
Other:
- note added: "There should be a 1 Ohm resistor between the emitter\nand ground here, but it's large enough as it is. Use\ntransistors somewhat equal to eachother. I'll add it to\nSMD-version if I get around to it. If in doubt, don't link\nthe pairs."
Changed lines of the file:
@@
 Text GLabel 1800 6725 1    50   Input ~ 0
 EX_B
+Wire Notes Line
+	2725 3075 4975 3075
+Wire Notes Line
+	4975 3075 4975 3150
+Wire Notes Line
+	4975 3150 2725 3150
+Text Notes 2800 3825 0    50   ~ 0
+There should be a 1 Ohm resistor between the emitter\nand ground here, but it's large enough as it is. Use\ntransistors somewhat equal to eachother. I'll add it to\nSMD-version if I get around to it. If in doubt, don't link\nthe pairs.
+Wire Notes Line
+	2725 3450 2775 3450
+Wire Notes Line
+	2725 3075 2725 3450
 $EndSCHEMATC
