File: RC Dashboard Digispark/RC Dashboard Digispark.kicad_pcb (KiCad board)
At the start: 2 copper layers, 25.2 x 24.1 mm, 10 parts, among them IC1 0.91_I2C_OLED, J5 THR, J6 THR_Y

Commit message: Small build tweaks to sizing and text
Routing:
- net /6v: track 53.3 -> 48.3 mm
- net Net-(A1-Pad8): track 21.5 -> 20.8 mm
Other:
- board size 25.2 x 24.1 mm -> 25.2 x 23.4 mm
- board text added: "RC Dashboard "Digispark" Rev. B"
- board text removed: "RC Dashboard "Digispark" Rev. A"
Changed lines of the file:
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@@
   (general
     (thickness 1.6)
-    (drawings 28)
-    (tracks 66)
+    (drawings 30)
+    (tracks 62)
     (zones 0)
     (modules 10)
@@
     )
   )
+  (gr_arc (start 100.772 78.74) (end 100.772 78.105) (angle -90) (layer Edge.Cuts) (width 0.05))
+  (gr_arc (start 124.75 78.74) (end 125.385 78.74) (angle -90) (layer Edge.Cuts) (width 0.05))
   (gr_text SDA (at 104.14 88.9 90) (layer F.SilkS)
     (effects (font (size 0.8 0.8) (thickness 0.1)))
@@
     (effects (font (size 0.8 0.8) (thickness 0.1)))
   )
-  (gr_line (start 125.385 77.47) (end 100.137 77.47) (layer Edge.Cuts) (width 0.05))
-  (gr_line (start 125.385 77.47) (end 125.382 97.441) (layer Edge.Cuts) (width 0.05))
+  (gr_line (start 124.75 78.105) (end 100.772 78.105) (layer Edge.Cuts) (width 0.05))
+  (gr_line (start 125.385 78.74) (end 125.382 97.441) (layer Edge.Cuts) (width 0.05))
   (gr_arc (start 121.282 97.441) (end 121.282 101.541) (angle -90) (layer Edge.Cuts) (width 0.05))
   (gr_arc (start 104.237 97.441) (end 100.137 97.441) (angle -90) (layer Edge.Cuts) (width 0.05))
-  (gr_line (start 100.137 97.441) (end 100.137 77.47) (layer Edge.Cuts) (width 0.05))
+  (gr_line (start 100.137 97.441) (end 100.137 78.74) (layer Edge.Cuts) (width 0.05))
   (gr_line (start 114.982 101.541) (end 121.282 101.541) (layer Edge.Cuts) (width 0.05))
   (gr_line (start 114.982 101.541) (end 104.237 101.541) (layer Edge.Cuts) (width 0.05))
@@
     (effects (font (size 0.8 0.8) (thickness 0.1)))
   )
-  (gr_text "RC Dashboard\n\"Digispark\"\nRev. A" (at 102.87 82.55 90) (layer F.SilkS)
+  (gr_text "RC Dashboard\n\"Digispark\"\nRev. B" (at 102.87 82.55 90) (layer F.SilkS)
     (effects (font (size 0.8 0.8) (thickness 0.1)))
   )
@@
   (segment (start 121.285 87.63) (end 121.285 90.17) (width 0.381) (layer F.Cu) (net 4))
   (segment (start 121.92 90.805) (end 123.751394 90.805) (width 0.381) (layer F.Cu) (net 4))
-  (segment (start 120.65 82.55) (end 116.205 82.55) (width 0.381) (layer F.Cu) (net 5))
   (via (at 114.3 82.55) (size 0.8) (drill 0.4) (layers F.Cu B.Cu) (net 5))
-  (segment (start 116.205 82.55) (end 114.3 82.55) (width 0.381) (layer F.Cu) (net 5))
   (segment (start 114.3 82.55) (end 114.3 81.28) (width 0.381) (layer B.Cu) (net 5))
   (segment (start 115.57 80.01) (end 116.205 80.01) (width 0.381) (layer B.Cu) (net 5) (status 30))
   (segment (start 114.3 81.28) (end 115.57 80.01) (width 0.381) (layer B.Cu) (net 5) (status 20))
-  (segment (start 120.65 82.55) (end 121.92 82.55) (width 0.381) (layer F.Cu) (net 5))
-  (segment (start 122.555 83.185) (end 122.555 84.455) (width 0.381) (layer F.Cu) (net 5))
-  (segment (start 121.92 82.55) (end 122.555 83.185) (width 0.381) (layer F.Cu) (net 5))
   (segment (start 109.22 80.01) (end 107.315 80.01) (width 0.381) (layer F.Cu) (net 5))
   (segment (start 111.76 82.55) (end 109.22 80.01) (width 0.381) (layer F.Cu) (net 5))
   (segment (start 114.3 82.55) (end 111.76 82.55) (width 0.381) (layer F.Cu) (net 5))
+  (segment (start 116.205 84.455) (end 114.3 82.55) (width 0.381) (layer F.Cu) (net 5))
+  (segment (start 122.555 84.455) (end 116.205 84.455) (width 0.381) (layer F.Cu) (net 5))
   (segment (start 102.235 93.98) (end 101.6 93.98) (width 0.381) (layer F.Cu) (net 6))
   (segment (start 101.6 93.98) (end 100.55251 92.93251) (width 0.381) (layer F.Cu) (net 6))
@@
   (segment (start 124.966515 97.283485) (end 124.968632 83.184982) (width 0.381) (layer F.Cu) (net 7))
   (segment (start 124.968632 83.184982) (end 124.968613 83.311386) (width 0.381) (layer F.Cu) (net 7))
-  (segment (start 124.968632 78.613632) (end 124.968632 83.184982) (width 0.381) (layer F.Cu) (net 7))
-  (segment (start 124.46 78.105) (end 124.968632 78.613632) (width 0.381) (layer F.Cu) (net 7))
-  (segment (start 113.03 78.105) (end 124.46 78.105) (width 0.381) (layer F.Cu) (net 7))
-  (segment (start 112.395 78.74) (end 113.03 78.105) (width 0.381) (layer F.Cu) (net 7))
-  (segment (start 112.395 80.01) (end 112.395 78.74) (width 0.381) (layer F.Cu) (net 7))
+  (segment (start 112.395 80.01) (end 115.57 80.01) (width 0.381) (layer F.Cu) (net 7))
+  (segment (start 115.57 80.01) (end 118.11 82.55) (width 0.381) (layer F.Cu) (net 7))
+  (segment (start 124.33365 82.55) (end 124.968632 83.184982) (width 0.381) (layer F.Cu) (net 7))
+  (segment (start 118.11 82.55) (end 124.33365 82.55) (width 0.381) (layer F.Cu) (net 7))
   (segment (start 106.045 92.71) (end 102.235 88.9) (width 0.381) (layer F.Cu) (net 8))
   (segment (start 109.855 92.71) (end 106.045 92.71) (width 0.381) (layer F.Cu) (net 8))
