File: RC Dashboard SuperMini2/RC Dashboard SuperMini2.kicad_pcb (KiCad board)
At the start: 2 copper layers, 26.3 x 33.2 mm, 16 parts, among them IC1 OLED, J1 LED1, J2 LED2, J5 CH1, J6 CH2, Q1 2N3904, Q2 2N3904

Commit message: SuperMini2
Parts:
- removed JP2: CFG1, solder_bridge:bridge
- JP3: value CFG2 -> CFG
Connections:
- net /CFG_2 renamed /CFG
- A1 pad 5: /CFG_1 -> unconnected-(A1-GPIO9-Pad5)
Routing:
- net /CFG_1: track 14.3 -> 0.00 mm
Changed lines of the file:
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@@
 	(net 6 "/BUILTIN_LED")
 	(net 7 "unconnected-(A1-GPIO6-Pad2)")
-	(net 8 "/CFG_1")
-	(net 9 "/CFG_2")
+	(net 8 "unconnected-(A1-GPIO9-Pad5)")
+	(net 9 "/CFG")
 	(net 10 "unconnected-(A1-GPIO21-Pad8)")
 	(net 11 "unconnected-(A1-GPIO4-Pad13)")
@@
 		)
 		(property "Value" "OLED"
-			(at 3.75 -1.7 270)
+			(at 3.75 -1.7 -90)
 			(unlocked yes)
 			(layer "B.SilkS")
@@
 		(tags "Resistor Axial_DIN0207 series Axial Horizontal pin pitch 7.62mm 0.25W = 1/4W length 6.3mm diameter 2.5mm")
 		(property "Reference" "R2"
-			(at 6.096 0 360)
+			(at 6.096 0 0)
 			(layer "F.SilkS")
 			(effects
@@
 		)
 		(fp_text user "${REFERENCE}"
-			(at 1.905 0 360)
+			(at 1.905 0 0)
 			(layer "F.Fab")
 			(effects
@@
 		)
 		(property "Value" "LED2"
-			(at 1.23 -1.7 270)
+			(at 1.23 -1.7 -90)
 			(unlocked yes)
 			(layer "B.SilkS")
@@
 		(tags "Resistor Axial_DIN0207 series Axial Horizontal pin pitch 7.62mm 0.25W = 1/4W length 6.3mm diameter 2.5mm")
 		(property "Reference" "R1"
-			(at 5.08 0 360)
+			(at 5.08 0 0)
 			(layer "F.SilkS")
 			(effects
@@
 		)
 		(fp_text user "${REFERENCE}"
-			(at 1.905 0 360)
+			(at 1.905 0 0)
 			(layer "F.Fab")
 			(effects
@@
 		(tags "Resistor Axial_DIN0207 series Axial Horizontal pin pitch 7.62mm 0.25W = 1/4W length 6.3mm diameter 2.5mm")
 		(property "Reference" "R4"
-			(at 6.096 0 360)
+			(at 6.096 0 0)
 			(layer "F.SilkS")
 			(effects
@@
 		)
 		(fp_text user "${REFERENCE}"
-			(at 1.905 0 360)
+			(at 1.905 0 0)
 			(layer "F.Fab")
 			(effects
@@
 		(tags "Resistor Axial_DIN0207 series Axial Horizontal pin pitch 7.62mm 0.25W = 1/4W length 6.3mm diameter 2.5mm")
 		(property "Reference" "R3"
-			(at 5.08 0 360)
+			(at 5.08 0 0)
 			(layer "F.SilkS")
 			(effects
@@
 		)
 		(fp_text user "${REFERENCE}"
-			(at 1.905 0 360)
+			(at 1.905 0 0)
 			(layer "F.Fab")
 			(effects
@@
 			(layers "*.Cu" "*.Mask")
 			(remove_unused_layers no)
-			(net 9 "/CFG_2")
+			(net 9 "/CFG")
 			(pinfunction "GPIO7")
 			(pintype "bidirectional")
@@
 			(layers "*.Cu" "*.Mask")
 			(remove_unused_layers no)
-			(net 8 "/CFG_1")
+			(net 8 "unconnected-(A1-GPIO9-Pad5)")
 			(pinfunction "GPIO9")
-			(pintype "bidirectional")
+			(pintype "bidirectional+no_connect")
 		)
 		(pad "6" thru_hole circle
@@
 	(footprint "solder_bridge:bridge"
 		(layer "B.Cu")
-		(at 106.045 75.8825 90)
-		(descr "Through hole straight pin header, 1x02, 1.00mm pitch, single row")
-		(tags "Through hole pin header THT 1x02 1.00mm single row")
-		(property "Reference" "JP2"
-			(at 0 2.54 90)
-			(layer "B.SilkS")
-			(hide yes)
-			(effects
-				(font
-					(size 1 1)
-					(thickness 0.15)
-				)
-				(justify mirror)
-			)
-		)
-		(property "Value" "CFG1"
-			(at 2.1717 -0.9398 0)
-			(unlocked yes)
-			(layer "B.SilkS")
-			(effects
-				(font
-					(size 0.8 0.8)
-					(thickness 0.1)
-				)
-				(justify mirror)
-			)
-		)
-		(property "Footprint" "solder_bridge:bridge"
-			(at 0 0 90)
-			(layer "B.Fab")
-			(hide yes)
-			(effects
-				(font
-					(size 1.27 1.27)
-					(thickness 0.15)
-				)
-				(justify mirror)
-			)
-		)
-		(property "Datasheet" ""
-			(at 0 0 90)
-			(layer "B.Fab")
-			(hide yes)
-			(effects
-				(font
-					(size 1.27 1.27)
-					(thickness 0.15)
-				)
-				(justify mirror)
-			)
-		)
-		(property "Description" "Jumper, 2-pole, open"
-			(at 0 0 90)
-			(layer "B.Fab")
-			(hide yes)
-			(effects
-				(font
-					(size 1.27 1.27)
-					(thickness 0.15)
-				)
-				(justify mirror)
-			)
-		)
-		(property ki_fp_filters "Jumper* TestPoint*2Pads* TestPoint*Bridge*")
-		(sheetname "Root")
-		(sheetfile "RC Dashboard SuperMini2.kicad_sch")
-		(attr through_hole)
-		(fp_line
-			(start 1.524 -3.175)
-			(end -1.524 -3.175)
-			(stroke
-				(width 0.15)
-				(type solid)
-			)
-			(layer "B.SilkS")
-		)
-		(fp_line
-			(start -1.524 -2.794)
-			(end -1.27 -2.794)
-			(stroke
-				(width 0.15)
-				(type solid)
-			)
-			(layer "B.SilkS")
-		)
-		(fp_line
-			(start -1.524 -2.794)
-			(end -1.524 0.762)
-			(stroke
-				(width 0.15)
-				(type solid)
-			)
-			(layer "B.SilkS")
-		)
-		(fp_line
-			(start -1.524 0.762)
-			(end -1.27 0.762)
-			(stroke
-				(width 0.15)
-				(type solid)
-			)
-			(layer "B.SilkS")
-		)
-		(fp_line
-			(start 1.524 1.27)
-			(end 1.524 -3.175)
-			(stroke
-				(width 0.15)
-				(type solid)
-			)
-			(layer "B.SilkS")
-		)
-		(fp_line
-			(start -1.524 1.27)
-			(end 1.524 1.27)
-			(stroke
-				(width 0.15)
-				(type solid)
-			)
-			(layer "B.SilkS")
-		)
-		(fp_text user "${REFERENCE}"
-			(at 0 -3.81 90)
-			(layer "B.Fab")
-			(effects
-				(font
-					(size 0.76 0.76)
-					(thickness 0.114)
-				)
-				(justify mirror)
-			)
-		)
-		(pad "1" smd rect
-			(at 0 0 90)
-			(size 2 1.5)
-			(layers "B.Cu" "B.Paste" "B.Mask")
-			(net 1 "GND")
-			(pinfunction "A")
-			(pintype "passive")
-		)
-		(pad "2" smd rect
-			(at 0 -1.905 90)
-			(size 2 1.5)
-			(layers "B.Cu" "B.Paste" "B.Mask")
-			(net 8 "/CFG_1")
-			(pinfunction "B")
-			(pintype "passive")
-		)
-		(model "${KISYS3DMOD}/Pin_Headers.3dshapes/Pin_Header_Straight_1x02_Pitch1.00mm.wrl"
-			(offset
-				(xyz 0 0 0)
-			)
-			(scale
-				(xyz 1 1 1)
-			)
-			(rotate
-				(xyz 0 0 0)
-			)
-		)
-	)
-	(footprint "solder_bridge:bridge"
-		(layer "B.Cu")
 		(at 106.045 79.6925 90)
 		(descr "Through hole straight pin header, 1x02, 1.00mm pitch, single row")
@@
 			)
 		)
-		(property "Value" "CFG2"
-			(at 0 1.905 270)
+		(property "Value" "CFG"
+			(at 2.2733 -0.9652 0)
 			(unlocked yes)
 			(layer "B.SilkS")
@@
 			(size 2 1.5)
 			(layers "B.Cu" "B.Paste" "B.Mask")
-			(net 9 "/CFG_2")
+			(net 9 "/CFG")
 			(pinfunction "B")
 			(pintype "passive")
@@
 	)
 	(segment
-		(start 99.695 84.455)
-		(end 100.0125 84.7725)
-		(width 0.25)
-		(layer "B.Cu")
-		(net 8)
-	)
-	(segment
-		(start 100.0125 84.7725)
-		(end 101.384184 84.7725)
-		(width 0.25)
-		(layer "B.Cu")
-		(net 8)
-	)
-	(segment
-		(start 100.6475 75.8825)
-		(end 99.695 76.835)
-		(width 0.25)
-		(layer "B.Cu")
-		(net 8)
-	)
-	(segment
-		(start 104.14 75.8825)
-		(end 100.6475 75.8825)
-		(width 0.25)
-		(layer "B.Cu")
-		(net 8)
-	)
-	(segment
-		(start 99.695 76.835)
-		(end 99.695 84.455)
-		(width 0.25)
-		(layer "B.Cu")
-		(net 8)
-	)
-	(segment

Commit message: Slight build tweaks
Parts:
- moved JP3 2.29 mm to (104.8, 77.8), turned to 180 degrees
Other:
- board text added: "Revision B github.com/tebl"
- board text removed: "Revision A github.com/tebl"
Changed lines of the file:
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@@
 	(footprint "solder_bridge:bridge"
 		(layer "B.Cu")
-		(at 106.045 79.6925 90)
+		(at 104.775 77.7875 180)
 		(descr "Through hole straight pin header, 1x02, 1.00mm pitch, single row")
 		(tags "Through hole pin header THT 1x02 1.00mm single row")
 		(property "Reference" "JP3"
-			(at 0 2.54 90)
+			(at 0 2.54 360)
 			(layer "B.SilkS")
 			(hide yes)
@@
 		)
 		(property "Value" "CFG"
-			(at 2.2733 -0.9652 0)
+			(at -2.413 -0.9525 -90)
 			(unlocked yes)
 			(layer "B.SilkS")
@@
 		)
 		(property "Footprint" "solder_bridge:bridge"
-			(at 0 0 90)
+			(at 0 0 360)
 			(layer "B.Fab")
 			(hide yes)
@@
 		)
 		(property "Datasheet" ""
-			(at 0 0 90)
+			(at 0 0 360)
 			(layer "B.Fab")
 			(hide yes)
@@
 		)
 		(property "Description" "Jumper, 2-pole, open"
-			(at 0 0 90)
+			(at 0 0 360)
 			(layer "B.Fab")
 			(hide yes)
@@
 		(attr through_hole)
 		(fp_line
+			(start 1.524 1.27)
+			(end 1.524 -3.175)
+			(stroke
+				(width 0.15)
+				(type solid)
+			)
+			(layer "B.SilkS")
+		)
+		(fp_line
 			(start 1.524 -3.175)
 			(end -1.524 -3.175)
@@
 		)
 		(fp_line
+			(start -1.524 1.27)
+			(end 1.524 1.27)
+			(stroke
+				(width 0.15)
+				(type solid)
+			)
+			(layer "B.SilkS")
+		)
+		(fp_line
+			(start -1.524 0.762)
+			(end -1.27 0.762)
+			(stroke
+				(width 0.15)
+				(type solid)
+			)
+			(layer "B.SilkS")
+		)
+		(fp_line
 			(start -1.524 -2.794)
 			(end -1.27 -2.794)
@@
 			(layer "B.SilkS")
 		)
-		(fp_line
-			(start -1.524 0.762)
-			(end -1.27 0.762)
-			(stroke
-				(width 0.15)
-				(type solid)
-			)
-			(layer "B.SilkS")
-		)
-		(fp_line
-			(start 1.524 1.27)
-			(end 1.524 -3.175)
-			(stroke
-				(width 0.15)
-				(type solid)
-			)
-			(layer "B.SilkS")
-		)
-		(fp_line
-			(start -1.524 1.27)
-			(end 1.524 1.27)
-			(stroke
-				(width 0.15)
-				(type solid)
-			)
-			(layer "B.SilkS")
-		)
 		(fp_text user "${REFERENCE}"
-			(at 0 1.5875 90)
+			(at 0 1.5875 360)
 			(layer "B.Fab")
 			(effects
@@
 		)
 		(pad "1" smd rect
-			(at 0 0 90)
+			(at 0 0 180)
 			(size 2 1.5)
 			(layers "B.Cu" "B.Paste" "B.Mask")
@@
 		)
 		(pad "2" smd rect
-			(at 0 -1.905 90)
+			(at 0 -1.905 180)
 			(size 2 1.5)
 			(layers "B.Cu" "B.Paste" "B.Mask")
@@
 	)
 	(gr_line
-		(start 104.559184 94.615)
-		(end 104.559184 94.615)
-		(stroke
-			(width 0.12)
-			(type default)
-		)
-		(layer "B.SilkS")
-	)
-	(gr_line
 		(start 106.68 99.695)
 		(end 106.68 99.695)
@@
 	)
 	(gr_line
-		(start 116.5105 104.9286)
-		(end 116.5105 104.4206)
+		(start 115.8755 104.9286)
+		(end 115.8755 104.4206)
 		(stroke
 			(width 0.12)
@@
 	)
 	(gr_line
-		(start 117.1455 104.9286)
-		(end 117.2725 104.9286)
-		(stroke
-			(width 0.12)
-			(type solid)
-		)
-		(layer "F.SilkS")
-	)
-	(gr_line
 		(start 116.5105 104.9286)
-		(end 116.3835 104.9286)
-		(stroke
-			(width 0.12)
-			(type solid)
-		)
-		(layer "F.SilkS")
-	)
-	(gr_line
-		(start 116.5105 104.4206)
-		(end 117.1455 104.4206)
+		(end 116.6375 104.9286)
+		(stroke
+			(width 0.12)
+			(type solid)
+		)
+		(layer "F.SilkS")
+	)
+	(gr_line
+		(start 115.8755 104.9286)
+		(end 115.7485 104.9286)
+		(stroke
+			(width 0.12)
+			(type solid)
+		)
+		(layer "F.SilkS")
+	)
+	(gr_line
+		(start 115.8755 104.4206)
+		(end 116.5105 104.4206)
 		(stroke
 			(width 0.12)
@@
 	)
 	(gr_line
-		(start 117.1455 104.4206)
-		(end 117.1455 104.9286)
+		(start 116.5105 104.4206)
+		(end 116.5105 104.9286)
 		(stroke
 			(width 0.12)
@@
 		)
 	)
-	(gr_text "Revision A\ngithub.com/tebl"
+	(gr_text "Revision B\ngithub.com/tebl"
 		(at 111.125 80.3 270)
 		(layer "B.SilkS")
@@
 	)
 	(gr_text "-"
-		(at 111.76 104.7635 180)
-		(layer "F.SilkS")
-		(effects
+		(at 111.125 104.7635 180)
+		(layer "F.SilkS")
+		(effects

Commit message: Missing track
Routing:
- net /CFG: track 2.76 -> 3.39 mm
Changed lines of the file:
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@@
 		(tags "Through hole pin header THT 1x02 1.00mm single row")
 		(property "Reference" "JP3"
-			(at 0 2.54 360)
+			(at 0 2.54 0)
 			(layer "B.SilkS")
 			(hide yes)
@@
 		)
 		(property "Footprint" "solder_bridge:bridge"
-			(at 0 0 360)
+			(at 0 0 0)
 			(layer "B.Fab")
 			(hide yes)
@@
 		)
 		(property "Datasheet" ""
-			(at 0 0 360)
+			(at 0 0 0)
 			(layer "B.Fab")
 			(hide yes)
@@
 		)
 		(property "Description" "Jumper, 2-pole, open"
-			(at 0 0 360)
+			(at 0 0 0)
 			(layer "B.Fab")
 			(hide yes)
@@
 		)
 		(fp_text user "${REFERENCE}"
-			(at 0 1.5875 360)
+			(at 0 1.5875 0)
 			(layer "B.Fab")
 			(effects
@@
 	)
 	(segment
-		(start 104.14 79.6925)
+		(start 104.775 79.6925)
 		(end 101.384184 79.6925)
 		(width 0.25)
