File: RC SCX10.3 Rock Control/RC SCX10.3 Rock Control.kicad_pcb (KiCad board)
At the start: 2 copper layers, 28.3 x 36.8 mm, 17 parts, among them J1 LED1, J2 LED2, J3 LED3, J4 LED4, J5 CH1, J6 CH2, Q1 2N2222, Q2 2N2222, Q3 2N2222, Q4 2N2222

Commit message: Small build tweaks
Parts:
- moved JP3 2.29 mm to (104.8, 77.8), turned to 180 degrees
Routing:
- net /CFG: track 2.76 -> 3.39 mm
Other:
- board text added: "6v"
Changed lines of the file:
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@@
 	(footprint "solder_bridge:bridge"
 		(layer "B.Cu")
-		(at 106.045 79.6925 90)
+		(at 104.775 77.7875 180)
 		(descr "Through hole straight pin header, 1x02, 1.00mm pitch, single row")
 		(tags "Through hole pin header THT 1x02 1.00mm single row")
 		(property "Reference" "JP3"
-			(at 0 2.54 90)
+			(at 0 2.54 360)
 			(layer "B.SilkS")
 			(hide yes)
@@
 		)
 		(property "Value" "CFG"
-			(at 0 1.905 -90)
+			(at -2.54 -0.9525 -90)
 			(unlocked yes)
 			(layer "B.SilkS")
@@
 		)
 		(property "Footprint" "solder_bridge:bridge"
-			(at 0 0 90)
+			(at 0 0 360)
 			(layer "B.Fab")
 			(hide yes)
@@
 		)
 		(property "Datasheet" ""
-			(at 0 0 90)
+			(at 0 0 360)
 			(layer "B.Fab")
 			(hide yes)
@@
 		)
 		(property "Description" "Jumper, 2-pole, open"
-			(at 0 0 90)
+			(at 0 0 360)
 			(layer "B.Fab")
 			(hide yes)
@@
 		(attr through_hole)
 		(fp_line
+			(start 1.524 1.27)
+			(end 1.524 -3.175)
+			(stroke
+				(width 0.15)
+				(type solid)
+			)
+			(layer "B.SilkS")
+		)
+		(fp_line
 			(start 1.524 -3.175)
 			(end -1.524 -3.175)
+			(stroke
+				(width 0.15)
+				(type solid)
+			)
+			(layer "B.SilkS")
+		)
+		(fp_line
+			(start -1.524 1.27)
+			(end 1.524 1.27)
+			(stroke
+				(width 0.15)
+				(type solid)
+			)
+			(layer "B.SilkS")
+		)
+		(fp_line
+			(start -1.524 0.762)
+			(end -1.27 0.762)
 			(stroke
 				(width 0.15)
@@
 			(layer "B.SilkS")
 		)
-		(fp_line
-			(start -1.524 0.762)
-			(end -1.27 0.762)
-			(stroke
-				(width 0.15)
-				(type solid)
-			)
-			(layer "B.SilkS")
-		)
-		(fp_line
-			(start 1.524 1.27)
-			(end 1.524 -3.175)
-			(stroke
-				(width 0.15)
-				(type solid)
-			)
-			(layer "B.SilkS")
-		)
-		(fp_line
-			(start -1.524 1.27)
-			(end 1.524 1.27)
-			(stroke
-				(width 0.15)
-				(type solid)
-			)
-			(layer "B.SilkS")
-		)
 		(fp_text user "${REFERENCE}"
-			(at 0 1.5875 90)
+			(at 0 1.5875 360)
 			(layer "B.Fab")
 			(effects
@@
 		)
 		(pad "1" smd rect
-			(at 0 0 90)
+			(at 0 0 180)
 			(size 2 1.5)
 			(layers "B.Cu" "B.Paste" "B.Mask")
@@
 		)
 		(pad "2" smd rect
-			(at 0 -1.905 90)
+			(at 0 -1.905 180)
 			(size 2 1.5)
 			(layers "B.Cu" "B.Paste" "B.Mask")
@@
 	)
 	(gr_line
-		(start 116.5105 108.7386)
-		(end 116.5105 108.2306)
+		(start 115.8748 108.712)
+		(end 115.8748 108.204)
 		(stroke
 			(width 0.12)
@@
 	)
 	(gr_line
-		(start 117.1455 108.7386)
-		(end 117.2725 108.7386)
-		(stroke
-			(width 0.12)
-			(type solid)
-		)
-		(layer "F.SilkS")
-	)
-	(gr_line
-		(start 116.5105 108.7386)
-		(end 116.3835 108.7386)
-		(stroke
-			(width 0.12)
-			(type solid)
-		)
-		(layer "F.SilkS")
-	)
-	(gr_line
-		(start 116.5105 108.2306)
-		(end 117.1455 108.2306)
+		(start 116.5098 108.712)
+		(end 116.6368 108.712)
+		(stroke
+			(width 0.12)
+			(type solid)
+		)
+		(layer "F.SilkS")
+	)
+	(gr_line
+		(start 115.8748 108.712)
+		(end 115.7478 108.712)
+		(stroke
+			(width 0.12)
+			(type solid)
+		)
+		(layer "F.SilkS")
+	)
+	(gr_line
+		(start 115.8748 108.204)
+		(end 116.5098 108.204)
 		(stroke
 			(width 0.12)
@@
 	)
 	(gr_line
-		(start 117.1455 108.2306)
-		(end 117.1455 108.7386)
+		(start 116.5098 108.204)
+		(end 116.5098 108.712)
 		(stroke
 			(width 0.12)
@@
 	)
 	(gr_text "+"
-		(at 114.3 108.5735 180)
+		(at 113.665 108.5735 180)
 		(layer "F.SilkS")
 		(effects
@@
 	)
 	(gr_text "-"
-		(at 111.76 108.5735 180)
+		(at 111.125 108.5735 180)
 		(layer "F.SilkS")
 		(effects
@@
 		)
 	)
+	(gr_text "-"
+		(at 96.52 75.565 0)
+		(layer "F.SilkS")
+		(effects
+			(font
+				(size 0.8 0.8)
+				(thickness 0.1)
+			)
+		)
+	)
+	(gr_text "6v"
+		(at 96.52 78.105 0)
+		(layer "F.SilkS")
+		(effects
+			(font
+				(size 0.8 0.8)
+				(thickness 0.1)
+			)
+		)
+	)
+	(gr_text "-"
+		(at 96.52 93.345 0)
+		(layer "F.SilkS")
+		(effects
+			(font
+				(size 0.8 0.8)
+				(thickness 0.1)
+			)
+		)
+	)
+	(gr_text "6v"
+		(at 96.52 95.885 0)
+		(layer "F.SilkS")
+		(effects
+			(font
+				(size 0.8 0.8)
+				(thickness 0.1)
+			)
+		)
+	)
+	(gr_text "6v"
+		(at 96.52 86.995 0)
+		(layer "F.SilkS")
+		(effects
+			(font
+				(size 0.8 0.8)
+				(thickness 0.1)
+			)
+		)
+	)
+	(gr_text "6v"
+		(at 96.52 104.775 0)
+		(layer "F.SilkS")
+		(effects
+			(font
+				(size 0.8 0.8)
+				(thickness 0.1)
+			)
+		)
+	)
 	(gr_text "WayWayWay"
 		(at 103.886 77.8256 90)
@@
 		)
 	)
+	(gr_text "-"
+		(at 96.52 84.455 0)
+		(layer "F.SilkS")
+		(effects
+			(font
+				(size 0.8 0.8)
+				(thickness 0.1)
+			)
+		)
+	)
+	(gr_text "-"
+		(at 96.52 102.235 0)
+		(layer "F.SilkS")
+		(effects
+			(font
+				(size 0.8 0.8)
+				(thickness 0.1)
+			)
+		)
+	)
 	(segment
 		(start 113.665 85.09)
@@
 	)
 	(segment
-		(start 104.14 79.6925)
+		(start 104.775 79.6925)
 		(end 101.384184 79.6925)
 		(width 0.25)
