File: RC Dashboard SuperMini/RC Dashboard SuperMini.kicad_pcb (KiCad board)
At the start: 2 copper layers, 26.3 x 27.2 mm, 8 parts, among them IC1 0.91_I2C_OLED, J5 CH1, J6 CH2

Commit message: Small build tweaks
Connections:
- net Net-(A1-GPIO0) renamed /SCL
- net Net-(A1-GPIO1) renamed /SDA
Routing:
- net /SDA: track 13.1 -> 13.9 mm
Changed lines of the file:
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@@
 	(net 0 "")
 	(net 1 "GND")
-	(net 2 "Net-(A1-GPIO1)")
-	(net 3 "Net-(A1-GPIO0)")
+	(net 2 "/SDA")
+	(net 3 "/SCL")
 	(net 4 "+3V3")
 	(net 5 "/6v")
@@
 			(layers "*.Cu" "*.Mask")
 			(remove_unused_layers no)
-			(net 3 "Net-(A1-GPIO0)")
+			(net 3 "/SCL")
 			(pinfunction "SCL")
 			(pintype "bidirectional")
@@
 			(layers "*.Cu" "*.Mask")
 			(remove_unused_layers no)
-			(net 2 "Net-(A1-GPIO1)")
+			(net 2 "/SDA")
 			(pinfunction "SDA")
 			(pintype "bidirectional")
@@
 			(layers "*.Cu" "*.Mask")
 			(remove_unused_layers no)
-			(net 3 "Net-(A1-GPIO0)")
+			(net 3 "/SCL")
 			(pinfunction "GPIO0")
 			(pintype "bidirectional")
@@
 			(layers "*.Cu" "*.Mask")
 			(remove_unused_layers no)
-			(net 2 "Net-(A1-GPIO1)")
+			(net 2 "/SDA")
 			(pinfunction "GPIO1")
 			(pintype "bidirectional")
@@
 	)
 	(gr_text "-"
-		(at 120.015 89.8652 -90)
+		(at 124.46 89.8652 -90)
 		(layer "B.SilkS")
 		(effects
@@
 	)
 	(gr_text "+"
-		(at 120.015 92.4052 -90)
+		(at 124.46 92.4052 -90)
 		(layer "B.SilkS")
 		(effects
@@
 	)
 	(gr_text "SCL"
-		(at 120.015 94.9452 -90)
+		(at 124.46 94.9452 -90)
 		(layer "B.SilkS")
 		(effects
@@
 	)
 	(gr_text "SDA"
-		(at 120.015 97.4852 -90)
+		(at 124.46 97.4852 -90)
 		(layer "B.SilkS")
 		(effects
@@
 	)
 	(segment
-		(start 116.84 94.9325)
-		(end 119.0625 94.9325)
+		(start 114.935 95.885)
+		(end 114.935 98.425)
 		(width 0.381)
 		(layer "F.Cu")
@@
 	)
 	(segment
-		(start 120.263 93.732)
-		(end 123.577 93.732)
+		(start 116.205 99.695)
+		(end 120.3325 99.695)
 		(width 0.381)
 		(layer "F.Cu")
@@
 	)
 	(segment
-		(start 123.577 93.732)
-		(end 124.46 94.615)
+		(start 116.84 94.9325)
+		(end 115.8875 94.9325)
 		(width 0.381)
 		(layer "F.Cu")
@@
 	)
 	(segment
-		(start 124.1425 97.4725)
+		(start 120.3325 99.695)
 		(end 122.555 97.4725)
 		(width 0.381)
@@
 	)
 	(segment
-		(start 119.0625 94.9325)
-		(end 120.263 93.732)
+		(start 114.935 98.425)
+		(end 116.205 99.695)
 		(width 0.381)
 		(layer "F.Cu")
@@
 	)
 	(segment
-		(start 124.46 94.615)
-		(end 124.46 97.155)
+		(start 115.8875 94.9325)
+		(end 114.935 95.885)
 		(width 0.381)
 		(layer "F.Cu")
-		(net 2)
-	)
-	(segment
-		(start 124.46 97.155)
-		(end 124.1425 97.4725)
-		(width 0.381)
-		(layer "F.Cu")

Commit message: Preparing for the next thing
Parts:
- JP1: value Y_CABLE -> 2CH
Connections:
- net Net-(A1-GPIO7) renamed /CFG_2
- net Net-(A1-GPIO9) renamed /CFG_1
- A1 pad 11: unconnected-(A1-GPIO2-Pad11) -> /LED_1
- A1 pad 12: unconnected-(A1-GPIO3-Pad12) -> /LED_2
- A1 pad 4: unconnected-(A1-GPIO8-Pad4) -> /BUILTIN_LED
Changed lines of the file:
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@@
 	(net 4 "+3V3")
 	(net 5 "/6v")
-	(net 6 "unconnected-(A1-GPIO2-Pad11)")
+	(net 6 "/BUILTIN_LED")
 	(net 7 "unconnected-(A1-GPIO6-Pad2)")
-	(net 8 "unconnected-(A1-GPIO3-Pad12)")
-	(net 9 "unconnected-(A1-GPIO8-Pad4)")
+	(net 8 "/CFG_1")
+	(net 9 "/CFG_2")
 	(net 10 "unconnected-(A1-GPIO21-Pad8)")
 	(net 11 "unconnected-(A1-GPIO4-Pad13)")
@@
 	(net 14 "CH1")
 	(net 15 "Net-(J5-VCC)")
-	(net 16 "Net-(A1-GPIO7)")
+	(net 16 "/LED_1")
 	(net 17 "VBUS")
-	(net 18 "Net-(A1-GPIO9)")
+	(net 18 "/LED_2")
 	(footprint "Diode_THT:D_DO-41_SOD81_P10.16mm_Horizontal"
 		(layer "F.Cu")
@@
 			(layers "*.Cu" "*.Mask")
 			(remove_unused_layers no)
-			(net 16 "Net-(A1-GPIO7)")
+			(net 9 "/CFG_2")
 			(pinfunction "GPIO7")
 			(pintype "bidirectional")
@@
 			(layers "*.Cu" "*.Mask")
 			(remove_unused_layers no)
-			(net 9 "unconnected-(A1-GPIO8-Pad4)")
+			(net 6 "/BUILTIN_LED")
 			(pinfunction "GPIO8")
 			(pintype "bidirectional+no_connect")
@@
 			(layers "*.Cu" "*.Mask")
 			(remove_unused_layers no)
-			(net 18 "Net-(A1-GPIO9)")
+			(net 8 "/CFG_1")
 			(pinfunction "GPIO9")
 			(pintype "bidirectional")
@@
 			(layers "*.Cu" "*.Mask")
 			(remove_unused_layers no)
-			(net 6 "unconnected-(A1-GPIO2-Pad11)")
+			(net 16 "/LED_1")
 			(pinfunction "GPIO2")
 			(pintype "bidirectional+no_connect")
@@
 			(layers "*.Cu" "*.Mask")
 			(remove_unused_layers no)
-			(net 8 "unconnected-(A1-GPIO3-Pad12)")
+			(net 18 "/LED_2")
 			(pinfunction "GPIO3")
 			(pintype "bidirectional+no_connect")
@@
 			(size 2 1.5)
 			(layers "B.Cu" "B.Paste" "B.Mask")
-			(net 18 "Net-(A1-GPIO9)")
+			(net 8 "/CFG_1")
 			(pinfunction "B")
 			(pintype "passive")
@@
 			(size 2 1.5)
 			(layers "B.Cu" "B.Paste" "B.Mask")
-			(net 16 "Net-(A1-GPIO7)")
+			(net 9 "/CFG_2")
 			(pinfunction "B")
 			(pintype "passive")
@@
 			)
 		)
-		(property "Value" "Y_CABLE"
+		(property "Value" "2CH"
 			(at 2.413 -1.9177 -90)
 			(unlocked yes)
@@
 	)
 	(segment
+		(start 103.1875 88.265)
+		(end 104.775 88.265)
+		(width 0.381)
+		(layer "B.Cu")
+		(net 8)
+	)
+	(segment
+		(start 101.6 89.8525)
+		(end 103.1875 88.265)
+		(width 0.381)
+		(layer "B.Cu")
+		(net 8)
+	)
+	(segment
+		(start 104.775 82.8675)
+		(end 103.505 82.8675)
+		(width 0.381)
+		(layer "B.Cu")
+		(net 9)
+	)
+	(segment
+		(start 103.505 82.8675)
+		(end 101.6 84.7725)
+		(width 0.381)
+		(layer "B.Cu")
+		(net 9)
+	)
+	(segment
 		(start 114.3 100.6475)
 		(end 116.205 102.5525)
@@
 	)
 	(segment
-		(start 104.775 82.8675)
-		(end 103.505 82.8675)
-		(width 0.381)
-		(layer "B.Cu")
-		(net 16)
-	)
-	(segment
-		(start 103.505 82.8675)
-		(end 101.6 84.7725)
-		(width 0.381)
-		(layer "B.Cu")
-		(net 16)
-	)
-	(segment
 		(start 112.395 82.2325)
 		(end 114.935 79.6925)
@@
 		(net 17)
 	)
-	(segment
-		(start 103.1875 88.265)
-		(end 104.775 88.265)
-		(width 0.381)
-		(layer "B.Cu")
-		(net 18)
-	)
-	(segment
-		(start 101.6 89.8525)
-		(end 103.1875 88.265)
-		(width 0.381)
-		(layer "B.Cu")
-		(net 18)
-	)
 	(zone

Commit message: Small build tweaks
Parts:
- removed JP2: CFG_1, solder_bridge:bridge
- JP3: value CFG_2 -> CFG
Connections:
- A1 pad 5: /CFG_1 -> unconnected-(A1-GPIO9-Pad5)
Routing:
- net /CFG_1: track 3.83 -> 0.00 mm
Other:
- board text added: "Dashboard {dblquote}SuperMini{dblquote} Rev. B"
- board text removed: "Dashboard {dblquote}SuperMini{dblquote} Rev. A"
Changed lines of the file:
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@@
 	(net 6 "/BUILTIN_LED")
 	(net 7 "unconnected-(A1-GPIO6-Pad2)")
-	(net 8 "/CFG_1")
+	(net 8 "unconnected-(A1-GPIO9-Pad5)")
 	(net 9 "/CFG_2")
 	(net 10 "unconnected-(A1-GPIO21-Pad8)")
@@
 			(layers "*.Cu" "*.Mask")
 			(remove_unused_layers no)
-			(net 8 "/CFG_1")
+			(net 8 "unconnected-(A1-GPIO9-Pad5)")
 			(pinfunction "GPIO9")
-			(pintype "bidirectional")
+			(pintype "bidirectional+no_connect")
 		)
 		(pad "6" thru_hole circle
@@
 			(pinfunction "5v")
 			(pintype "power_in")
-		)
-	)
-	(footprint "solder_bridge:bridge"
-		(layer "B.Cu")
-		(at 104.775 86.36 180)
-		(descr "Through hole straight pin header, 1x02, 1.00mm pitch, single row")
-		(tags "Through hole pin header THT 1x02 1.00mm single row")
-		(property "Reference" "JP2"
-			(at 0 2.54 0)
-			(layer "B.SilkS")
-			(hide yes)
-			(effects
-				(font
-					(size 1 1)
-					(thickness 0.15)
-				)
-				(justify mirror)
-			)
-		)
-		(property "Value" "CFG_1"
-			(at -2.413 -0.9144 -90)
-			(unlocked yes)
-			(layer "B.SilkS")
-			(effects
-				(font
-					(size 0.8 0.8)
-					(thickness 0.1)
-				)
-				(justify mirror)
-			)
-		)
-		(property "Footprint" "solder_bridge:bridge"
-			(at 0 0 0)
-			(layer "B.Fab")
-			(hide yes)
-			(effects
-				(font
-					(size 1.27 1.27)
-					(thickness 0.15)
-				)
-				(justify mirror)
-			)
-		)
-		(property "Datasheet" ""
-			(at 0 0 0)
-			(layer "B.Fab")
-			(hide yes)
-			(effects
-				(font
-					(size 1.27 1.27)
-					(thickness 0.15)
-				)
-				(justify mirror)
-			)
-		)
-		(property "Description" "Jumper, 2-pole, open"
-			(at 0 0 0)
-			(layer "B.Fab")
-			(hide yes)
-			(effects
-				(font
-					(size 1.27 1.27)
-					(thickness 0.15)
-				)
-				(justify mirror)
-			)
-		)
-		(property ki_fp_filters "Jumper* TestPoint*2Pads* TestPoint*Bridge*")
-		(sheetname "Root")
-		(sheetfile "RC Dashboard SuperMini.kicad_sch")
-		(attr through_hole)
-		(fp_line
-			(start 1.524 1.27)
-			(end 1.524 -3.175)
-			(stroke
-				(width 0.15)
-				(type solid)
-			)
-			(layer "B.SilkS")
-		)
-		(fp_line
-			(start 1.524 -3.175)
-			(end -1.524 -3.175)
-			(stroke
-				(width 0.15)
-				(type solid)
-			)
-			(layer "B.SilkS")
-		)
-		(fp_line
-			(start -1.524 1.27)
-			(end 1.524 1.27)
-			(stroke
-				(width 0.15)
-				(type solid)
-			)
-			(layer "B.SilkS")
-		)
-		(fp_line
-			(start -1.524 0.762)
-			(end -1.27 0.762)
-			(stroke
-				(width 0.15)
-				(type solid)
-			)
-			(layer "B.SilkS")
-		)
-		(fp_line
-			(start -1.524 -2.794)
-			(end -1.27 -2.794)
-			(stroke
-				(width 0.15)
-				(type solid)
-			)
-			(layer "B.SilkS")
-		)
-		(fp_line
-			(start -1.524 -2.794)
-			(end -1.524 0.762)
-			(stroke
-				(width 0.15)
-				(type solid)
-			)
-			(layer "B.SilkS")
-		)
-		(fp_text user "${REFERENCE}"
-			(at 0 -3.81 0)
-			(layer "B.Fab")
-			(effects
-				(font
-					(size 0.76 0.76)
-					(thickness 0.114)
-				)
-				(justify mirror)
-			)
-		)
-		(pad "1" smd rect
-			(at 0 0 180)
-			(size 2 1.5)
-			(layers "B.Cu" "B.Paste" "B.Mask")
-			(net 1 "GND")
-			(pinfunction "A")
-			(pintype "passive")
-		)
-		(pad "2" smd rect
-			(at 0 -1.905 180)
-			(size 2 1.5)
-			(layers "B.Cu" "B.Paste" "B.Mask")
-			(net 8 "/CFG_1")
-			(pinfunction "B")
-			(pintype "passive")
-		)
-		(model "${KISYS3DMOD}/Pin_Headers.3dshapes/Pin_Header_Straight_1x02_Pitch1.00mm.wrl"
-			(offset
-				(xyz 0 0 0)
-			)
-			(scale
-				(xyz 1 1 1)
-			)
-			(rotate
-				(xyz 0 0 0)
-			)
 		)
 	)
@@
 			)
 		)
-		(property "Value" "CFG_2"
+		(property "Value" "CFG"
 			(at -2.413 -0.9144 -90)
 			(unlocked yes)
@@
 	)
 	(gr_line
-		(start 116.5105 104.9286)
-		(end 116.5105 104.4206)
+		(start 115.8755 104.9286)
+		(end 115.8755 104.4206)
 		(stroke
 			(width 0.12)
@@
 	)
 	(gr_line
-		(start 117.1455 104.9286)
-		(end 117.2725 104.9286)
+		(start 116.5105 104.9286)
+		(end 116.6375 104.9286)
 		(stroke
 			(width 0.12)
@@
 	)
 	(gr_line
-		(start 116.5105 104.9286)
-		(end 116.3835 104.9286)
+		(start 115.8755 104.9286)
+		(end 115.7485 104.9286)
 		(stroke
 			(width 0.12)
@@
 	)
 	(gr_line
-		(start 116.5105 104.4206)
-		(end 117.1455 104.4206)
+		(start 115.8755 104.4206)
+		(end 116.5105 104.4206)
 		(stroke
 			(width 0.12)
@@
 	)
 	(gr_line
-		(start 117.1455 104.4206)
-		(end 117.1455 104.9286)
+		(start 116.5105 104.4206)
+		(end 116.5105 104.9286)
 		(stroke
 			(width 0.12)
@@
 	)
 	(gr_text "+"
-		(at 114.3 104.7635 180)
+		(at 113.665 104.7635 180)
 		(layer "F.SilkS")
 		(effects
@@
 	)
 	(gr_text "-"
-		(at 111.76 104.7635 180)
+		(at 111.125 104.7635 180)
 		(layer "F.SilkS")
 		(effects
@@
 		)
 	)
-	(gr_text "Dashboard\n{dblquote}SuperMini{dblquote}\nRev. A"
+	(gr_text "Dashboard\n{dblquote}SuperMini{dblquote}\nRev. B"
 		(at 118.11 102.616 0)
 		(layer "F.SilkS")
@@
 	)
 	(segment
-		(start 103.1875 88.265)
-		(end 104.775 88.265)
-		(width 0.381)
-		(layer "B.Cu")
-		(net 8)
-	)
-	(segment
-		(start 101.6 89.8525)
-		(end 103.1875 88.265)
-		(width 0.381)
-		(layer "B.Cu")
-		(net 8)
-	)
-	(segment
