File: RC Dashboard SuperMini/RC Dashboard SuperMini.kicad_sch (KiCad schematic)
At the start: 8 parts, among them IC1 0.91_I2C_OLED, J5 CH1, J6 CH2

Commit message: Small build tweaks
Connections:
- net SCL: now reaches A1.9 (GPIO0), IC1.3 (SCL)
- net SDA: now reaches A1.10 (GPIO1), IC1.4 (SDA)
Changed lines of the file:
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@@
+		)
+	)
+	(label "SCL"
+		(at 223.52 120.65 180)
+		(fields_autoplaced yes)
+		(effects
+			(font
+				(size 1.27 1.27)
+			)
+			(justify right bottom)
 		)
 	)
@@
 		)
 	)
+	(label "SDA"
+		(at 223.52 118.11 180)
+		(fields_autoplaced yes)
+		(effects
+			(font
+				(size 1.27 1.27)
+			)
+			(justify right bottom)
+		)
+	)

Commit message: Preparing for the next thing
Parts:
- JP1: value Y_CABLE -> 2CH
Connections:
- net CFG_2: now reaches A1.3 (GPIO7), JP3.2 (B)
- net LED_1: now reaches A1.11 (GPIO2)
- net LED_2: now reaches A1.12 (GPIO3)
- net BUILTIN_LED: now reaches A1.4 (GPIO8)
- net CFG_1: now reaches A1.5 (GPIO9), JP2.2 (B)
Other:
- moved on the sheet: JP2, JP3
Changed lines of the file:
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@@
 	)
 	(junction
-		(at 132.08 88.9)
+		(at 121.92 88.9)
 		(diameter 0)
 		(color 0 0 0 0)
@@
 	)
 	(no_connect
-		(at 200.66 91.44)
+		(at 217.17 88.9)
 	)
 	(no_connect
@@
 	)
 	(no_connect
-		(at 160.02 86.36)
+		(at 146.05 86.36)
 	)
 	(no_connect
@@
 	)
 	(no_connect
-		(at 200.66 88.9)
+		(at 217.17 91.44)
 	)
 	(wire
@@
 	(wire
 		(pts
+			(xy 200.66 88.9) (xy 217.17 88.9)
+		)
+		(stroke
+			(width 0)
+			(type default)
+		)
+	)
+	(wire
+		(pts
 			(xy 66.04 93.98) (xy 66.04 102.87)
 		)
@@
 	(wire
 		(pts
-			(xy 156.21 91.44) (xy 160.02 91.44)
-		)
-		(stroke
-			(width 0)
-			(type default)
-		)
-	)
-	(wire
-		(pts
 			(xy 66.04 83.82) (xy 66.04 93.98)
 		)
@@
 	(wire
 		(pts
-			(xy 132.08 88.9) (xy 137.16 88.9)
-		)
-		(stroke
-			(width 0)
-			(type default)
-		)
-	)
-	(wire
-		(pts
-			(xy 132.08 83.82) (xy 137.16 83.82)
-		)
-		(stroke
-			(width 0)
-			(type default)
-		)
-	)
-	(wire
-		(pts
-			(xy 132.08 83.82) (xy 132.08 88.9)
-		)
-		(stroke
-			(width 0)
-			(type default)
-		)
-	)
-	(wire
-		(pts
-			(xy 156.21 93.98) (xy 160.02 93.98)
+			(xy 121.92 88.9) (xy 127 88.9)
+		)
+		(stroke
+			(width 0)
+			(type default)
+		)
+	)
+	(wire
+		(pts
+			(xy 121.92 83.82) (xy 127 83.82)
+		)
+		(stroke
+			(width 0)
+			(type default)
+		)
+	)
+	(wire
+		(pts
+			(xy 121.92 83.82) (xy 121.92 88.9)
 		)
 		(stroke
@@
 	(wire
 		(pts
+			(xy 137.16 88.9) (xy 160.02 88.9)
+		)
+		(stroke
+			(width 0)
+			(type default)
+		)
+	)
+	(wire
+		(pts
 			(xy 71.12 71.12) (xy 71.12 73.66)
 		)
@@
 	(wire
 		(pts
-			(xy 132.08 88.9) (xy 132.08 96.52)
+			(xy 121.92 88.9) (xy 121.92 96.52)
 		)
 		(stroke
@@
 	(wire
 		(pts
+			(xy 137.16 83.82) (xy 160.02 83.82)
+		)
+		(stroke
+			(width 0)
+			(type default)
+		)
+	)
+	(wire
+		(pts
 			(xy 63.5 86.36) (xy 59.69 86.36)
 		)
@@
 	(wire
 		(pts
-			(xy 147.32 88.9) (xy 160.02 88.9)
+			(xy 146.05 91.44) (xy 160.02 91.44)
+		)
+		(stroke
+			(width 0)
+			(type default)
+		)
+	)
+	(wire
+		(pts
+			(xy 146.05 93.98) (xy 160.02 93.98)
 		)
 		(stroke
@@
 	(wire
 		(pts
+			(xy 146.05 86.36) (xy 160.02 86.36)
+		)
+		(stroke
+			(width 0)
+			(type default)
+		)
+	)
+	(wire
+		(pts
 			(xy 208.28 125.73) (xy 208.28 128.27)
 		)
@@
 	(wire
 		(pts
-			(xy 147.32 83.82) (xy 160.02 83.82)
-		)
-		(stroke
-			(width 0)
-			(type default)
-		)
-	)
-	(wire
-		(pts
 			(xy 215.9 118.11) (xy 224.79 118.11)
+		)
+		(stroke
+			(width 0)
+			(type default)
+		)
+	)
+	(wire
+		(pts
+			(xy 200.66 91.44) (xy 217.17 91.44)
 		)
 		(stroke
@@
 		)
 	)
+	(label "CFG_2"
+		(at 147.32 83.82 0)
+		(fields_autoplaced yes)
+		(effects
+			(font
+				(size 1.27 1.27)
+			)
+			(justify left bottom)
+		)
+	)
+	(label "LED_1"
+		(at 215.9 91.44 180)
+		(fields_autoplaced yes)
+		(effects
+			(font
+				(size 1.27 1.27)
+			)
+			(justify right bottom)
+		)
+	)
+	(label "CFG_1"
+		(at 147.32 88.9 0)
+		(fields_autoplaced yes)
+		(effects
+			(font
+				(size 1.27 1.27)
+			)
+			(justify left bottom)
+		)
+	)
 	(label "SCL"
 		(at 223.52 120.65 180)
@@
 		)
 	)
+	(label "LED_2"
+		(at 215.9 88.9 180)
+		(fields_autoplaced yes)
+		(effects
+			(font
+				(size 1.27 1.27)
+			)
+			(justify right bottom)
+		)
+	)
 	(label "SDA"
 		(at 223.52 118.11 180)
@@
 		)
 	)
+	(label "BUILTIN_LED"
+		(at 158.75 86.36 180)
+		(fields_autoplaced yes)
+		(effects
+			(font
+				(size 1.27 1.27)
+			)
+			(justify right bottom)
+		)
+	)
 	(global_label "CH1"
 		(shape output)
@@
 	(global_label "CH2"
 		(shape input)
-		(at 156.21 91.44 180)
+		(at 146.05 91.44 180)
 		(effects
 			(font
@@
 		)
 		(property "Intersheetrefs" "${INTERSHEET_REFS}"
-			(at 156.21 91.44 0)
+			(at 146.05 91.44 0)
 			(effects
 				(font
@@
 	(global_label "CH1"
 		(shape input)
-		(at 156.21 93.98 180)
+		(at 146.05 93.98 180)
 		(effects
 			(font
@@
 		)
 		(property "Intersheetrefs" "${INTERSHEET_REFS}"
-			(at 156.21 93.98 0)
+			(at 146.05 93.98 0)
 			(effects
 				(font
@@
 			)
 		)
-		(property "Value" "Y_CABLE"
+		(property "Value" "2CH"
 			(at 80.01 87.63 0)
 			(effects
@@
 	(symbol
 		(lib_id "power:GND")
-		(at 132.08 96.52 0)
+		(at 121.92 96.52 0)
 		(unit 1)
 		(exclude_from_sim no)
@@
 		(fields_autoplaced yes)
 		(property "Reference" "#PWR02"
-			(at 132.08 102.87 0)
+			(at 121.92 102.87 0)
 			(effects
 				(font
@@
 		)
 		(property "Value" "GND"
-			(at 132.08 101.6 0)
+			(at 121.92 101.6 0)
 			(effects
 				(font
@@
 		)
 		(property "Footprint" ""
-			(at 132.08 96.52 0)
+			(at 121.92 96.52 0)
 			(effects
 				(font
@@
 		)
 		(property "Datasheet" ""
-			(at 132.08 96.52 0)
+			(at 121.92 96.52 0)
 			(effects
 				(font
@@
 		)
 		(property "Description" "Power symbol creates a global label with name \"GND\" , ground"
-			(at 132.08 96.52 0)
+			(at 121.92 96.52 0)
 			(effects
 				(font
@@
 	(symbol
 		(lib_id "Jumper:Jumper_2_Open")
-		(at 142.24 83.82 0)
+		(at 132.08 83.82 0)
 		(unit 1)
 		(exclude_from_sim yes)
@@
 		(dnp no)
 		(property "Reference" "JP3"
-			(at 142.24 77.47 0)
+			(at 132.08 77.47 0)
 			(effects
 				(font
@@
 		)
 		(property "Value" "CFG_2"
-			(at 142.24 80.01 0)
+			(at 132.08 80.01 0)
 			(effects
 				(font
@@
 		)
 		(property "Footprint" "solder_bridge:bridge"
-			(at 142.24 83.82 0)
+			(at 132.08 83.82 0)
 			(effects
 				(font
@@
 		)
 		(property "Datasheet" "~"
-			(at 142.24 83.82 0)
+			(at 132.08 83.82 0)
 			(effects
 				(font
@@
 		)
 		(property "Description" "Jumper, 2-pole, open"
-			(at 142.24 83.82 0)
+			(at 132.08 83.82 0)
 			(effects
 				(font
@@
 		(on_board yes)
 		(dnp no)
-		(fields_autoplaced yes)
 		(property "Reference" "#PWR03"
 			(at 208.28 72.39 0)
@@
 		)
 		(property "Value" "+3V3"
-			(at 208.28 63.5 0)
+			(at 208.28 62.23 0)
 			(effects
 				(font
@@
 	(symbol
 		(lib_id "Jumper:Jumper_2_Open")
-		(at 142.24 88.9 0)
+		(at 132.08 88.9 0)
 		(mirror x)
 		(unit 1)
@@
 		(dnp no)
 		(property "Reference" "JP2"
-			(at 142.24 92.71 0)
+			(at 132.08 92.71 0)
 			(effects
 				(font
@@
 		)
 		(property "Value" "CFG_1"
-			(at 142.24 95.25 0)
+			(at 132.08 95.25 0)
 			(effects
 				(font
@@
 		)
 		(property "Footprint" "solder_bridge:bridge"
-			(at 142.24 88.9 0)
+			(at 132.08 88.9 0)
 			(effects
 				(font
@@
 		)
 		(property "Datasheet" "~"
-			(at 142.24 88.9 0)
+			(at 132.08 88.9 0)
 			(effects
 				(font
@@
 		)
 		(property "Description" "Jumper, 2-pole, open"
-			(at 142.24 88.9 0)
+			(at 132.08 88.9 0)
 			(effects
 				(font
@@
 		(on_board yes)
 		(dnp no)
-		(fields_autoplaced yes)
 		(property "Reference" "#PWR07"
 			(at 204.47 72.39 0)
@@
 		)
 		(property "Value" "VBUS"
-			(at 204.47 63.5 0)
-			(effects
-				(font
+			(at 204.47 64.77 0)
+			(effects
+				(font

Commit message: Small build tweaks
Parts:
- removed JP2: CFG_1, solder_bridge:bridge, symbol Jumper:Jumper_2_Open
- JP3: value CFG_2 -> CFG
Connections:
- net CFG_1 renamed BOOT
- net CFG_2 renamed CFG
- no-connect marks 7 -> 8
Changed lines of the file:
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@@
-	)
-	(junction
-		(at 121.92 88.9)
-		(diameter 0)
-		(color 0 0 0 0)
 	)
 	(junction
@@
 	)
 	(no_connect
+		(at 146.05 88.9)
+	)
+	(no_connect
 		(at 160.02 81.28)
 	)
@@
 	(wire
 		(pts
-			(xy 121.92 88.9) (xy 127 88.9)
-		)
-		(stroke
-			(width 0)
-			(type default)
-		)
-	)
-	(wire
-		(pts
 			(xy 121.92 83.82) (xy 127 83.82)
 		)
@@
 	(wire
 		(pts
-			(xy 121.92 83.82) (xy 121.92 88.9)
+			(xy 121.92 83.82) (xy 121.92 96.52)
 		)
 		(stroke
@@
 	(wire
 		(pts
-			(xy 137.16 88.9) (xy 160.02 88.9)
-		)
-		(stroke
-			(width 0)
-			(type default)
-		)
-	)
-	(wire
-		(pts
 			(xy 71.12 71.12) (xy 71.12 73.66)
 		)
@@
 	(wire
 		(pts
-			(xy 121.92 88.9) (xy 121.92 96.52)
-		)
-		(stroke
-			(width 0)
-			(type default)
-		)
-	)
-	(wire
-		(pts
 			(xy 204.47 68.58) (xy 204.47 78.74)
 		)
@@
 		(pts
 			(xy 208.28 125.73) (xy 208.28 128.27)
+		)
+		(stroke
+			(width 0)
+			(type default)
+		)
+	)
+	(wire
+		(pts
+			(xy 146.05 88.9) (xy 160.02 88.9)
 		)
 		(stroke
@@
 		)
 	)
-	(label "CFG_2"
+	(label "BOOT"
+		(at 147.32 88.9 0)
+		(fields_autoplaced yes)
+		(effects
+			(font
+				(size 1.27 1.27)
+			)
+			(justify left bottom)
+		)
+	)
+	(label "CFG"
 		(at 147.32 83.82 0)
 		(fields_autoplaced yes)
@@
 		)
 	)
-	(label "CFG_1"
-		(at 147.32 88.9 0)
-		(fields_autoplaced yes)
-		(effects
-			(font
-				(size 1.27 1.27)
-			)
-			(justify left bottom)
-		)
-	)
 	(label "SCL"
 		(at 223.52 120.65 180)
@@
 	)
 	(label "BUILTIN_LED"
-		(at 158.75 86.36 180)
+		(at 147.32 86.36 0)
 		(fields_autoplaced yes)
 		(effects
@@
 				(size 1.27 1.27)
 			)
-			(justify right bottom)
+			(justify left bottom)
 		)
 	)
@@
 			)
 		)
-		(property "Value" "CFG_2"
+		(property "Value" "CFG"
 			(at 132.08 80.01 0)
 			(effects
@@
 					(unit 1)
 				)
-			)
-		)
-	)
-	(symbol
-		(lib_id "Jumper:Jumper_2_Open")
-		(at 132.08 88.9 0)
-		(mirror x)
-		(unit 1)
-		(exclude_from_sim yes)
-		(in_bom yes)
-		(on_board yes)
-		(dnp no)
-		(property "Reference" "JP2"
-			(at 132.08 92.71 0)
-			(effects
-				(font
-					(size 1.27 1.27)
-				)
-			)
-		)
-		(property "Value" "CFG_1"
-			(at 132.08 95.25 0)
-			(effects
-				(font
-					(size 1.27 1.27)
-				)
-			)
-		)
-		(property "Footprint" "solder_bridge:bridge"
-			(at 132.08 88.9 0)
-			(effects
-				(font
-					(size 1.27 1.27)
-				)
-				(hide yes)
-			)
-		)
-		(property "Datasheet" "~"
-			(at 132.08 88.9 0)
-			(effects
-				(font
-					(size 1.27 1.27)
-				)
-				(hide yes)
-			)
-		)
-		(property "Description" "Jumper, 2-pole, open"
-			(at 132.08 88.9 0)
-			(effects
-				(font
-					(size 1.27 1.27)
-				)
-				(hide yes)
-			)
-		)
-		(pin "1"
-		)
-		(pin "2"
-		)
-		(instances
-			(project ""
-				(path "/8ea515ea-bab1-45cc-8dd8-41301b605afe"
-					(reference "JP2")
-					(unit 1)
-				)
